File: hardware/PCB/main_pcb.kicad_pcb (KiCad board)
At the start: 2 copper layers, 50 x 50 mm, 7 parts

Commit message: update,
Parts:
- removed the REF** at (100.0, 35.4)
- removed the REF** at (85.4, 45.0)
- added REF**: Val**, 2EDGK.pretty:degson-2EDGR-5.08-02P-14-00AH-0-0-0, F.Cu at (129.0, 37.0)
- added REF**: Val**, 2EDGK.pretty:degson-2EDGR-5.08-02P-14-00AH-0-0-0, F.Cu at (145.0, 37.0)
- added REF**: ESP32-WROOM-32D, ESP32-WROOM-32D:ESP32-WROOM-32D, F.Cu at (112.0, 61.0)
- added REF**: DC_JACK, DC_JACK:DC_JACK, F.Cu at (112.0, 44.0)
- added REF**: USBC_16PIN, footprint:USBC_16PIN, F.Cu at (98.0, 35.4)
- added REF**: USBC_16PIN, footprint:USBC_16PIN, F.Cu at (85.0, 64.0)
- moved REF** 36.1 mm to (155.0, 65.0)
- moved H2 30.0 mm to (155.0, 35.0)
- moved H4 30.0 mm to (155.0, 75.0)
Other:
- board size 50 x 50 mm -> 80 x 50 mm

Commit message: update,
Parts:
- removed the REF** at (129.0, 37.0)
- removed the REF** at (145.0, 37.0)
- removed the REF** at (98.0, 35.4)
- removed the REF** at (85.0, 64.0)
- removed the REF** at (155.0, 65.0)
- added REF**: Val**, 2EDGV:2EDGV-5.08-02P, F.Cu at (145.5, 40.0)
- added REF**: Val**, 2EDGV:2EDGV-5.08-02P, F.Cu at (134.5, 40.0)
- added REF**: TTL_TERMINAL_2.54mm, footprint:TTL_TERMINAL_2.54mm, F.Cu at (156.0, 62.0)
- added REF**: USBC_16PIN, footprint:USBC_16PIN, F.Cu at (98.0, 33.5)
- moved REF** 16.8 mm to (96.0, 56.0), turned to 90 degrees
- moved REF** 4.00 mm to (112.0, 40.0)

Commit message: update,
Parts:
- added REF**: CP_Elec_10x10, Capacitor_SMD:CP_Elec_10x10, F.Cu at (119.5, 52.0)
